Commit message: able to grasp the chess sets rn

File: ur_robot_env/urdf/simple_gripper.xacro (robot description, xacro)
@@ -12,5 +12,4 @@
       <visual>
         <origin xyz="0 0 0" rpy="0 0 0"/>
-        <!-- 使用圓柱體讓外型看起來較精緻 -->
         <geometry>
           <cylinder length="0.02" radius="0.01"/>
@@ -44,5 +43,5 @@
         <origin xyz="0.04 0 0" rpy="0 0 0"/>
         <geometry>
-          <box size="0.08 0.015 0.04"/>
+          <box size="0.08 0.006 0.076"/>
         </geometry>
         <material name="Blue">
@@ -53,5 +52,5 @@
         <origin xyz="0.04 0 0" rpy="0 0 0"/>
         <geometry>
-          <box size="0.08 0.015 0.04"/>
+          <box size="0.08 0.006 0.076"/>
         </geometry>
         <surface>
@@ -72,5 +71,5 @@
         <origin xyz="0.04 0 0" rpy="0 0 0"/>
         <geometry>
-          <box size="0.08 0.015 0.04"/>
+          <box size="0.075 0.006 0.076"/>
         </geometry>
         <material name="Blue">
@@ -81,5 +80,5 @@
         <origin xyz="0.04 0 0" rpy="0 0 0"/>
         <geometry>
-          <box size="0.08 0.015 0.04"/>
+          <box size="0.08 0.006 0.076"/>
         </geometry>
         <surface>
